File: LICHEE-JACK_EXT_BOARD.kicad_pcb (KiCad board)
At the start: 4 copper layers, 45.6 x 28 mm, 39 parts, among them J1 ETH100M_1-2, J2 ETH100M_3-6, J3 ETH100M-1236, Q1 AO3401A, Q2 AO3401A, Q3 AO3400, Q4 AO3400, U1 TP5400, U2 LM66100DCKR, U3 LicheeRV_Nano

Commit message: v1.1
Parts:
- removed the G*** at (82.8, 60.9)
- added D5: SS1X-323, PMEG4010CEJ_115:DIO_PMEG4010CEJ_115, B.Cu at (90.8, 84.5)
- added G***: LOGO, UUID:8e5ac303-e0d3-4627-85d2-c048de4b0b68, B.Cu at (82.8, 60.9)
Connections:
- S2 pad 2: GPIO_16 -> GPIO_15
Routing:
- net GPIO_16: track 12.2 -> 0.00 mm, vias 2 -> 0
- net GPIO_15: track 0.00 -> 9.53 mm, vias 0 -> 2
- net PWR_IN: track 59.9 -> 65.8 mm
- net PWR_OUT: track 55.0 -> 60.1 mm
Other:
- board text added: "8e5ac303-e0d3-4627-85d2-c048de4b0b68"
- board text added: "Lichee-Jack EXT. board v1.1"
- board text removed: "Lichee-Jack EXT. board v1.0"
- board text removed: "e4de6107-d49f-4286-95e3-404f75bb2bef"
