File: LICHEE-JACK_EXT_BOARD.kicad_sch (KiCad schematic)
At the start: 33 parts, among them J1 ETH100M_1-2, J2 ETH100M_3-6, J3 ETH100M-1236, Q1 AO3401A, Q2 AO3401A, Q3 AO3400, Q4 AO3400, U1 TP5400, U2 LM66100DCKR, U3 LicheeRV_Nano

Commit message: v1.1
Parts:
- added D5: SS1X-323, PMEG4010CEJ_115:DIO_PMEG4010CEJ_115, symbol PMEG4010CEJ_115:PMEG4010CEJ_115
Connections:
- net PWR_IN: now also D5.2
- net PWR_OUT: now also D5.1
- net GPIO_16 renamed GPIO_15
- net GPIO_15: now also U3.4 (GPIOA_15); no longer U3.2 (GPIOA_16/UART0_TX/PWM_4)
